Commit message: 使用修正的urdf

File: env/linghou_description/urdf/LingHouUrdf3.urdf (robot description, URDF)
Before this commit: robot LR4_R560, 16 links, 15 joints
Links:
- link LR4_R560_link2_respondable: geometry collision mesh filename=../meshes/linkhou_LR4_R560_link2_respondable_coll_1.dae; collision mesh filename=../meshes/linkhou_LR4_R560_link2_respondable_coll_10.dae
- link LR4_R560_link3_respondable: geometry collision mesh filename=../meshes/linkhou_LR4_R560_link3_respondable_coll_1.dae; collision mesh filename=../meshes/linkhou_LR4_R560_link3_respondable_coll_10.dae
- link LR4_R560_link4_respondable: geometry collision mesh filename=../meshes/linkhou_LR4_R560_link4_respondable_coll_1.dae; collision mesh filename=../meshes/linkhou_LR4_R560_link4_respondable_coll_10.dae
- link LR4_R560_link5_respondable: geometry collision mesh filename=../meshes/linkhou_LR4_R560_link5_respondable_coll_1.dae; collision mesh filename=../meshes/linkhou_LR4_R560_link5_respondable_coll_10.dae
- link LR4_R560_link6_respondable: geometry collision mesh filename=../meshes/linkhou_LR4_R560_link6_respondable_coll_1.dae; collision mesh filename=../meshes/linkhou_LR4_R560_link6_respondable_coll_10.dae
- link LR4_R560_link7_respondable: geometry collision mesh filename=../meshes/linkhou_LR4_R560_link7_respondable_coll_1.dae; collision mesh filename=../meshes/linkhou_LR4_R560_link7_respondable_coll_10.dae
- link left_finger_respondable: geometry collision mesh filename=../meshes/linkhou_left_finger_respondable_coll_1.dae; visual mesh filename=../meshes/linkhou_left_finger_visual_vis_1.dae
- link left_inner_knuckle_respondable: geometry collision mesh filename=../meshes/linkhou_left_inner_knuckle_respondable_coll_1.dae; visual mesh filename=../meshes/linkhou_left_inner_knuckle_visual_vis_1.dae
- link left_outer_knuckle_respondable: geometry collision mesh filename=../meshes/linkhou_left_outer_knuckle_respondable_coll_1.dae; visual mesh filename=../meshes/linkhou_left_outer_knuckle_visual_vis_1.dae
- link right_finger_respondable: geometry collision mesh filename=../meshes/linkhou_right_finger_respondable_coll_1.dae; visual mesh filename=../meshes/linkhou_right_finger_visual_vis_1.dae
- link right_inner_knuckle_respondable: geometry collision mesh filename=../meshes/linkhou_right_inner_knuckle_respondable_coll_1.dae; visual mesh filename=../meshes/linkhou_right_inner_knuckle_visual_vis_1.dae
- link right_outer_knuckle_respondable: geometry collision mesh filename=../meshes/linkhou_right_outer_knuckle_respondable_coll_1.dae; visual mesh filename=../meshes/linkhou_right_outer_knuckle_visual_vis_1.dae
- link robot_base: geometry collision mesh filename=../meshes/linkhou_robot_base_coll_1.dae; collision mesh filename=../meshes/linkhou_robot_base_coll_10.dae
- link xarm_gripper_base_link_respondable: geometry collision mesh filename=../meshes/linkhou_xarm_gripper_base_link_respondable_coll_1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; visual mesh filename=../meshes/linkhou_xarm_gripper_base_link_visual_vis_1.dae
Joints:
- joint LR4_R560_joint1: origin xyz=-0.05145 -0.00004 0.20057 rpy=-3.14160 3.14160 3.14160 -> xyz=0.090228 -0.000044 0.200573 rpy=-3.141589 3.141593 3.141593
- joint LR4_R560_joint2: origin xyz=-0.02000 -0.00000 0.14450 rpy=-1.57080 3.14159 -3.14159 -> xyz=-0.020000 -0.000000 0.144500 rpy=-1.570800 3.141593 -3.141592
- joint LR4_R560_joint3: origin xyz=0.00000 0.26000 0.00000 rpy=-3.14159 3.14160 -0.00000 -> xyz=0.000000 0.260000 0.000000 rpy=-3.141592 3.141600 -0.000000
- joint LR4_R560_joint4: origin xyz=0.09018 -0.01915 0.00000 rpy=-1.57079 3.14160 -1.56141 -> xyz=0.090184 -0.019152 0.000000 rpy=-1.570785 3.141592 -1.561411
- joint LR4_R560_joint5: origin xyz=0.00000 0.00000 0.19000 rpy=-1.57047 1.58018 -3.14127 -> xyz=0.000002 0.000000 0.190000 rpy=-1.570471 1.580184 -3.141265
- joint LR4_R560_joint6: origin xyz=-0.06700 0.00063 -0.00000 rpy=1.57079 3.14159 -1.58019 -> xyz=-0.066997 0.000631 -0.000000 rpy=1.570791 2.181661 -1.580196
- joint drive_joint: origin xyz=-0.059098 0.035000 -0.000000 rpy=-3.141593 3.141593 -3.141593 -> xyz=-0.059098 0.035000 -0.000000 rpy=-3.141593 3.141593 3.141593
- joint gripper_fix: origin xyz=0.000000 0.000000 0.000000 rpy=3.141593 3.141593 3.141593 -> xyz=0.000000 0.000000 0.000000 rpy=-3.141593 3.141593 -3.141593
- joint joint_eef: origin xyz=-0.00015 0.00013 0.00526 rpy=-3.13438 1.59529 3.06020 -> xyz=-0.000154 0.000131 0.005256 rpy=-2.316304 1.571449 1.567710
- joint joint_tcp: origin xyz=-0.172000 -0.000000 -0.000000 rpy=-3.141593 3.141593 -3.141593 -> xyz=-0.172000 0.000000 -0.000000 rpy=-3.141593 3.141593 3.141593
- joint left_inner_knuckle_joint: origin xyz=-0.074098 0.020000 -0.000000 rpy=-3.141593 3.141593 -3.141593 -> xyz=-0.074098 0.020000 -0.000000 rpy=-3.141593 3.141593 3.141593

Commit message: urdf删除惯性相关数据

File: env/linghou_description/urdf/LingHouUrdf3.urdf (robot description, URDF)
Before this commit: robot LR4_R560, 16 links, 15 joints
Links:
- link LR4_R560_link2_respondable: mass 6.0 -> None
- link LR4_R560_link3_respondable: mass 5.0 -> None
- link LR4_R560_link4_respondable: mass 2.0 -> None
- link LR4_R560_link5_respondable: mass 1.5 -> None
- link LR4_R560_link6_respondable: mass 1.2 -> None
- link LR4_R560_link7_respondable: mass 0.3 -> None
- link left_finger_respondable: mass 0.048304 -> None
- link left_inner_knuckle_respondable: mass 0.023012578125671 -> None
- link left_outer_knuckle_respondable: mass 0.033618 -> None
- link right_finger_respondable: mass 0.048304 -> None
- link right_inner_knuckle_respondable: mass 0.023013 -> None
- link right_outer_knuckle_respondable: mass 0.033618 -> None
- link robot_base: mass 10.0 -> None
- link xarm_gripper_base_link_respondable: mass 0.54156 -> None

Commit message: 训练成功率提高

File: env/linghou_description/urdf/LingHouUrdf3.urdf (robot description, URDF)
Before this commit: robot LR4_R560, 16 links, 15 joints
Links:
- link LR4_R560_link2_respondable: mass 6.0 -> None
- link LR4_R560_link3_respondable: mass 5.0 -> None
- link LR4_R560_link4_respondable: mass 2.0 -> None
- link LR4_R560_link5_respondable: mass 1.5 -> None
- link LR4_R560_link6_respondable: mass 1.2 -> None
- link LR4_R560_link7_respondable: mass 0.3 -> None
- link robot_base: mass 10.0 -> None

Commit message: 关节角度限制

File: env/linghou_description/urdf/LingHouUrdf3.urdf (robot description, URDF)
Before this commit: robot LR4_R560, 16 links, 15 joints
Joints:
- joint LR4_R560_joint1: limit lower=-2.967 upper=2.967 effort=23.0 velocity=7.255 -> lower=-2.932 upper=2.932 effort=23.0 velocity=7.255
- joint LR4_R560_joint2: limit lower=-2.495 upper=1.518 effort=23.0 velocity=7.255 -> lower=-1.570 upper=2.094 effort=23.0 velocity=7.255
- joint LR4_R560_joint3: limit lower=-3.577 upper=0.925 effort=20.7 velocity=8.062 -> lower=-1.57 upper=0.925 effort=20.7 velocity=8.062
- joint LR4_R560_joint4: limit lower=-3.490 upper=3.490 effort=16.3 velocity=8.727 -> lower=-2.967 upper=2.967 effort=16.3 velocity=8.727

Commit message: 轨迹回放、夹爪偏移、夹爪模型修改、夹取角度修改

File: env/linghou_description/urdf/LingHouUrdf3.urdf (robot description, URDF)
Before this commit: robot LR4_R560, 16 links, 15 joints
Links:
- link xarm_gripper_base_link_respondable: geometry collision mesh filename=../meshes/linkhou_xarm_gripper_base_link_respondable_coll_1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; visual mesh filename=../meshes/linkhou_xarm_gripper_base_link_visual_vis_1.dae scale=1 1 1
Joints:
- joint LR4_R560_joint2: limit lower=-1.570 upper=2.094 effort=23.0 velocity=7.255 -> lower=-1.517 upper=2.094 effort=23.0 velocity=7.255
- joint drive_joint: limit lower=0.0 upper=0.85 effort=50.0 velocity=2.0 -> lower=0.0 upper=0.65 effort=50.0 velocity=2.0
- joint right_outer_knuckle_joint: limit lower=0.0 upper=0.85 effort=50.0 velocity=2.0 -> lower=0.0 upper=0.65 effort=50.0 velocity=2.0
